File: schema/piecyk.sch (KiCad schematic (older format))
At the start: 30 parts, among them IC1 ATMEGA8-AI, P1 PWR_IN, P2 PWR_OUT, P3 CONN_01X04, P4 CONN_01X04, P5 ISP_IDC, Q1 2N7002, Q2 2N7002, Q3 BC516, SW1 SW_edit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

Commit message: Add missing pull-down resistor, adjust brightness levels
Parts:
- added R8: 10k, Resistors_SMD:R_0805_HandSoldering, symbol R
Connections:
- net GND: now also R8.1
- net LCD_Blight_PWM: now also R8.2
Changed lines of the file:
@@
 	0    -1   1    0
 $EndComp
+$Comp
+L R R8
+U 1 1 548D650C
+P 7200 1550
+F 0 "R8" V 7280 1550 40  0000 C CNN
+F 1 "10k" V 7207 1551 40  0000 C CNN
+F 2 "Resistors_SMD:R_0805_HandSoldering" V 7130 1550 30  0001 C CNN
+F 3 "" H 7200 1550 30  0000 C CNN
+	1    7200 1550
+	0    1    1    0
+$EndComp
+Wire Wire Line
+	7450 1550 7950 1550
+Connection ~ 7950 1550
+Wire Wire Line
+	6950 1550 6850 1550
+Wire Wire Line
+	6850 1550 6850 1250
+Connection ~ 6850 1250
 $EndSCHEMATC
